File: spaceduino-dummy-experiment/spaceduino.kicad_pcb (KiCad board)
At the start: 2 copper layers, 69 x 69 mm, 72 parts, among them J1 USB_B, J3 JICSP, J4 Conn_02x05_Odd_Even, Q1 BSS84, Q2 BSS84, Q3 BSS84, SW1 SW_SPST, U1 TLV70030_SOT23-5, U2 FT230XS, U3 TXB0104D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

Commit message: dummy experiment versions, set up .gitignore
Parts:
- added U8: MPD200A, Spaceduino:MPD200A, B.Cu at (97.1, 71.0)
Connections:
- J4 pad 5: Net-(J4-Pad5) -> pump+
- J4 pad 9: Net-(J4-Pad9) -> pump-
Routing:
- net pump-: track 0.00 -> 29.7 mm
- net 23: track 0.00 -> 24.3 mm, vias 0 -> 2
- net pump+: track 0.00 -> 16.1 mm
