File: containment-simple/containment-simple.sch (KiCad schematic (older format))
At the start: 26 parts

Commit message: containment simple mostly done
Parts:
- removed D? (x3): LED, symbol Device:LED
- removed J?: Conn_01x12, symbol Connector_Generic:Conn_01x12
- removed JP? (x8): Jumper, symbol Device:Jumper_NO_Small
- removed Q? (x3): BSS84, Package_TO_SOT_SMD:SOT-23, symbol Transistor_FET:BSS84
- removed R? (x3): 1k, symbol Device:R
- removed U?: PCF8574, symbol Interface_Expansion:PCF8574
- added C1: .1uF, Capacitor_SMD:C_0603_1608Metric, symbol Device:C
- added C3: 10uF, Capacitor_SMD:C_1206_3216Metric, symbol Device:C
- added D2, D4, D6, D8: D, Diode_SMD:D_SOD-123, symbol Device:D
- added D5, D7, D9: LED, LED_SMD:LED_1206_3216Metric, symbol Device:LED
- added H1, H2, H3, H4: MountingHole_Pad, Containment:MountingHole_2-56_ExtraClearance, symbol Mechanical:MountingHole_Pad
- added J1: Conn_02x05_Odd_Even, Connector_PinHeader_2.54mm:PinHeader_2x05_P2.54mm_Vertical, symbol Connector_Generic:Conn_02x05_Odd_Even
- added J3, J4, J5, J6: Conn_01x02, Connector_PinHeader_2.54mm:PinHeader_1x02_P2.54mm_Vertical, symbol Connector_Generic:Conn_01x02
- added Q2, Q3, Q4: BSS84, Package_TO_SOT_SMD:SOT-23, symbol Transistor_FET:BSS84
- added R3, R4, R5: 1k, Resistor_SMD:R_1206_3216Metric, symbol Device:R
- added U2: PCA9557, Package_SO:SOIC-16_3.9x9.9mm_P1.27mm, symbol Containment:PCA9557
- D1, D3: renamed from D?; footprint (none) -> LED_SMD:LED_1206_3216Metric
- JTEMP1: renamed from J?; value JTEMP -> Conn_01x02; footprint (none) -> Connector_PinHeader_2.54mm:PinHeader_1x02_P2.54mm_Vertical
- R1, R2: renamed from R?; footprint (none) -> Resistor_SMD:R_1206_3216Metric
- U1: renamed from U?; footprint (none) -> Package_SO:SOIC-8_3.9x4.9mm_P1.27mm
- gave numbers to parts that had none: 1
Connections:
- net +12V: now also J1.6 (Pin_6), Q3.2 (S), Q4.2 (S)
- net +5V: now also Q1.2 (S), C1.1, C3.1, J1.8 (Pin_8), Q2.2 (S), U2.15 (~RESET), U2.16 (VCC)
- net GND: now also C1.2, C3.2, D2.2 (A), D4.2 (A), D5.1 (K), D6.2 (A), D7.1 (K), D8.2 (A), D9.1 (K), H1.1, H2.1, H3.1, H4.1, J1.10 (Pin_10), J3.2 (Pin_2), J4.2 (Pin_2), J5.2 (Pin_2), J6.2 (Pin_2), U2.3 (A0), U2.4 (A1), U2.5 (A2), U2.8 (GND)
- net p0: now also U2.6 (P0); no longer Q1.1 (G)
- net p1: now also U2.7 (P1)
- net p2: now also U2.9 (P2)
- net p3: now also U2.10 (P3)
- net p4: now also Q1.1 (G), U2.11 (P4)
- net p5: now also Q2.1 (G), U2.12 (P5)
- net p6: now also Q3.1 (G), U2.13 (P6)
- net p7: now also Q4.1 (G), U2.14 (P7)
- net scl: now also J1.4 (Pin_4), U2.1 (SCL)
- net sda: now also J1.2 (Pin_2), U2.2 (SDA)
- net m0: no longer names the net of Q1.3 (D), R2.1
- net m0: now also D2.1 (K), J3.1 (Pin_1)
- new net: D4.1 (K), J4.1 (Pin_1), Q2.3 (D), R3.1
- new net: D5.2 (A), R3.2
- new net: D6.1 (K), J5.1 (Pin_1), Q3.3 (D), R4.1
- new net: D7.2 (A), R4.2
- new net: D8.1 (K), J6.1 (Pin_1), Q4.3 (D), R5.1
- new net: D9.2 (A), R5.2
- no-connect marks 0 -> 5

Commit message: some lcsc stuff
Parts:
- added R6, R7, R8, R9: 10k, Resistor_SMD:R_1206_3216Metric, symbol Device:R
Connections:
- net +5V: now also R6.1, R7.1, R8.1, R9.1
- net p4: now also R6.2
- net p5: now also R7.2
- net p6: now also R8.2
- net p7: now also R9.2
Changed lines of the file:
@@
 $EndComp
 Connection ~ 1450 1600
+$Comp
+L Device:R R6
+U 1 1 5F867E39
+P 4250 1250
+F 0 "R6" H 4320 1296 50  0000 L CNN
+F 1 "10k" H 4320 1205 50  0000 L CNN
+F 2 "Resistor_SMD:R_1206_3216Metric" V 4180 1250 50  0001 C CNN
+F 3 "~" H 4250 1250 50  0001 C CNN
+	1    4250 1250
+	1    0    0    -1
+$EndComp
+$Comp
+L Device:R R7
+U 1 1 5F86830F
+P 4500 1250
+F 0 "R7" H 4570 1296 50  0000 L CNN
+F 1 "10k" H 4570 1205 50  0000 L CNN
+F 2 "Resistor_SMD:R_1206_3216Metric" V 4430 1250 50  0001 C CNN
+F 3 "~" H 4500 1250 50  0001 C CNN
+	1    4500 1250
+	1    0    0    -1
+$EndComp
+$Comp
+L Device:R R8
+U 1 1 5F868690
+P 4750 1250
+F 0 "R8" H 4820 1296 50  0000 L CNN
+F 1 "10k" H 4820 1205 50  0000 L CNN
+F 2 "Resistor_SMD:R_1206_3216Metric" V 4680 1250 50  0001 C CNN
+F 3 "~" H 4750 1250 50  0001 C CNN
+	1    4750 1250
+	1    0    0    -1
+$EndComp
+$Comp
+L Device:R R9
+U 1 1 5F868C72
+P 5000 1250
+F 0 "R9" H 5070 1296 50  0000 L CNN
+F 1 "10k" H 5070 1205 50  0000 L CNN
+F 2 "Resistor_SMD:R_1206_3216Metric" V 4930 1250 50  0001 C CNN
+F 3 "~" H 5000 1250 50  0001 C CNN
+	1    5000 1250
+	1    0    0    -1
+$EndComp
+$Comp
+L power:+5V #PWR0122
+U 1 1 5F87145D
+P 4250 1100
+F 0 "#PWR0122" H 4250 950 50  0001 C CNN
+F 1 "+5V" H 4265 1273 50  0000 C CNN
+F 2 "" H 4250 1100 50  0001 C CNN
+F 3 "" H 4250 1100 50  0001 C CNN
+	1    4250 1100
+	1    0    0    -1
+$EndComp
+$Comp
+L power:+5V #PWR0124
+U 1 1 5F87199F
+P 4500 1100
+F 0 "#PWR0124" H 4500 950 50  0001 C CNN
+F 1 "+5V" H 4515 1273 50  0000 C CNN
+F 2 "" H 4500 1100 50  0001 C CNN
+F 3 "" H 4500 1100 50  0001 C CNN
+	1    4500 1100
+	1    0    0    -1
+$EndComp
+$Comp
+L power:+5V #PWR0125
+U 1 1 5F871CD6
+P 4750 1100
+F 0 "#PWR0125" H 4750 950 50  0001 C CNN
+F 1 "+5V" H 4765 1273 50  0000 C CNN
+F 2 "" H 4750 1100 50  0001 C CNN
+F 3 "" H 4750 1100 50  0001 C CNN
+	1    4750 1100
+	1    0    0    -1
+$EndComp
+$Comp
+L power:+5V #PWR0126
+U 1 1 5F8720DE
+P 5000 1100
+F 0 "#PWR0126" H 5000 950 50  0001 C CNN
+F 1 "+5V" H 5015 1273 50  0000 C CNN
+F 2 "" H 5000 1100 50  0001 C CNN
+F 3 "" H 5000 1100 50  0001 C CNN
+	1    5000 1100
+	1    0    0    -1
+$EndComp
+Wire Wire Line
+	4250 1400 4250 1800
+Wire Wire Line
+	4250 1800 4100 1800
+Wire Wire Line
+	4100 1900 4500 1900
+Wire Wire Line
+	4500 1900 4500 1400
+Wire Wire Line
+	4750 1400 4750 2000
+Wire Wire Line
+	4750 2000 4100 2000
+Wire Wire Line
+	4100 2100 5000 2100
+Wire Wire Line
+	5000 2100 5000 1400
 $EndSCHEMATC

Commit message: more lcsc, redo a lot of inner containment
Parts:
- C1: LCSC (none) -> C77055
- C3: LCSC (none) -> C14860
- D1, D3, D5, D7, D9: LCSC (none) -> C264549
- D2, D4, D6, D8: LCSC (none) -> C222352
- Q1, Q2, Q3, Q4: LCSC (none) -> C508197
- R1, R2, R3, R4, R5: footprint Resistor_SMD:R_1206_3216Metric -> Resistor_SMD:R_0603_1608Metric; LCSC (none) -> C50069
- R6, R7, R8, R9: footprint Resistor_SMD:R_1206_3216Metric -> Resistor_SMD:R_0603_1608Metric; LCSC (none) -> C491175
- U1: footprint Package_SO:SOIC-8_3.9x4.9mm_P1.27mm -> Package_SO:VSSOP-8_3.0x3.0mm_P0.65mm; LCSC (none) -> C475495
- U2: footprint Package_SO:SOIC-16_3.9x9.9mm_P1.27mm -> Package_SO:TSSOP-16_4.4x5mm_P0.65mm; LCSC (none) -> C141380
Changed lines of the file:
@@
 F 2 "Package_TO_SOT_SMD:SOT-23" H 6000 1075 50  0001 L CIN
 F 3 "http://assets.nexperia.com/documents/data-sheet/BSS84.pdf" H 5800 1150 50  0001 L CNN
+F 4 "C508197" H 5800 1150 50  0001 C CNN "LCSC"
 	1    5800 1150
 	1    0    0    1
@@
 F 0 "R1" H 920 3146 50  0000 L CNN
 F 1 "1k" H 920 3055 50  0000 L CNN
-F 2 "Resistor_SMD:R_1206_3216Metric" V 780 3100 50  0001 C CNN
+F 2 "Resistor_SMD:R_0603_1608Metric" V 780 3100 50  0001 C CNN
 F 3 "~" H 850 3100 50  0001 C CNN
+F 4 "C50069" H 850 3100 50  0001 C CNN "LCSC"
 	1    850  3100
 	1    0    0    -1
@@
 F 2 "LED_SMD:LED_1206_3216Metric" H 850 3400 50  0001 C CNN
 F 3 "~" H 850 3400 50  0001 C CNN
+F 4 "C264549" H 850 3400 50  0001 C CNN "LCSC"
 	1    850  3400
 	0    -1   -1   0
@@
 F 0 "U1" H 1550 5750 50  0000 C CNN
 F 1 "TMP411" H 1550 5650 50  0000 C CNN
-F 2 "Package_SO:SOIC-8_3.9x4.9mm_P1.27mm" H 1750 5200 50  0001 C CIN
+F 2 "Package_SO:VSSOP-8_3.0x3.0mm_P0.65mm" H 1750 5200 50  0001 C CIN
 F 3 "http://www.ti.com.cn/cn/lit/ds/symlink/tmp411.pdf" H 1750 5200 50  0001 C CNN
+F 4 "C475495" H 1850 5200 50  0001 C CNN "LCSC"
 	1    1850 5200
 	1    0    0    -1
@@
 F 2 "Diode_SMD:D_SOD-123" H 5900 1600 50  0001 C CNN
 F 3 "~" H 5900 1600 50  0001 C CNN
+F 4 "C222352" H 5900 1600 50  0001 C CNN "LCSC"
 	1    5900 1600
 	0    1    1    0
@@
 Connection ~ 1700 1700
 $Comp
-L Transistor_FET:BSS84 Q2
-U 1 1 5F26623C
-P 7250 1200
-F 0 "Q2" H 7454 1154 50  0000 L CNN
-F 1 "BSS84" H 7454 1245 50  0000 L CNN
-F 2 "Package_TO_SOT_SMD:SOT-23" H 7450 1125 50  0001 L CIN
-F 3 "http://assets.nexperia.com/documents/data-sheet/BSS84.pdf" H 7250 1200 50  0001 L CNN
-	1    7250 1200
-	1    0    0    1
-$EndComp
-$Comp
 L power:+5V #PWR0116
 U 1 1 5F266259
@@
 F 0 "R3" H 7770 1596 50  0000 L CNN
 F 1 "1k" H 7770 1505 50  0000 L CNN
-F 2 "Resistor_SMD:R_1206_3216Metric" V 7630 1550 50  0001 C CNN
+F 2 "Resistor_SMD:R_0603_1608Metric" V 7630 1550 50  0001 C CNN
 F 3 "~" H 7700 1550 50  0001 C CNN
+F 4 "C50069" H 7700 1550 50  0001 C CNN "LCSC"
 	1    7700 1550
 	1    0    0    -1
@@
 F 2 "LED_SMD:LED_1206_3216Metric" H 7700 1850 50  0001 C CNN
 F 3 "~" H 7700 1850 50  0001 C CNN
+F 4 "C264549" H 7700 1850 50  0001 C CNN "LCSC"
 	1    7700 1850
 	0    -1   -1   0
@@
 F 2 "Diode_SMD:D_SOD-123" H 7350 1650 50  0001 C CNN
 F 3 "~" H 7350 1650 50  0001 C CNN
+F 4 "C222352" H 7350 1650 50  0001 C CNN "LCSC"
 	1    7350 1650
 	0    1    1    0
@@
 F 2 "Package_TO_SOT_SMD:SOT-23" H 8800 1125 50  0001 L CIN
 F 3 "http://assets.nexperia.com/documents/data-sheet/BSS84.pdf" H 8600 1200 50  0001 L CNN
+F 4 "C508197" H 8600 1200 50  0001 C CNN "LCSC"
 	1    8600 1200
 	1    0    0    1
@@
 F 0 "R4" H 9120 1596 50  0000 L CNN
 F 1 "1k" H 9120 1505 50  0000 L CNN
-F 2 "Resistor_SMD:R_1206_3216Metric" V 8980 1550 50  0001 C CNN
+F 2 "Resistor_SMD:R_0603_1608Metric" V 8980 1550 50  0001 C CNN
 F 3 "~" H 9050 1550 50  0001 C CNN
+F 4 "C50069" H 9050 1550 50  0001 C CNN "LCSC"
 	1    9050 1550
 	1    0    0    -1
@@
 F 2 "LED_SMD:LED_1206_3216Metric" H 9050 1850 50  0001 C CNN
 F 3 "~" H 9050 1850 50  0001 C CNN
+F 4 "C264549" H 9050 1850 50  0001 C CNN "LCSC"
 	1    9050 1850
 	0    -1   -1   0
@@
 F 2 "Diode_SMD:D_SOD-123" H 8700 1650 50  0001 C CNN
 F 3 "~" H 8700 1650 50  0001 C CNN
+F 4 "C222352" H 8700 1650 50  0001 C CNN "LCSC"
 	1    8700 1650
 	0    1    1    0
@@
 F 2 "Package_TO_SOT_SMD:SOT-23" H 10150 1125 50  0001 L CIN
 F 3 "http://assets.nexperia.com/documents/data-sheet/BSS84.pdf" H 9950 1200 50  0001 L CNN
+F 4 "C508197" H 9950 1200 50  0001 C CNN "LCSC"
 	1    9950 1200
 	1    0    0    1
@@
 F 0 "R5" H 10470 1596 50  0000 L CNN
 F 1 "1k" H 10470 1505 50  0000 L CNN
-F 2 "Resistor_SMD:R_1206_3216Metric" V 10330 1550 50  0001 C CNN
+F 2 "Resistor_SMD:R_0603_1608Metric" V 10330 1550 50  0001 C CNN
 F 3 "~" H 10400 1550 50  0001 C CNN
+F 4 "C50069" H 10400 1550 50  0001 C CNN "LCSC"
 	1    10400 1550
 	1    0    0    -1
@@
 F 2 "LED_SMD:LED_1206_3216Metric" H 10400 1850 50  0001 C CNN
 F 3 "~" H 10400 1850 50  0001 C CNN
+F 4 "C264549" H 10400 1850 50  0001 C CNN "LCSC"
 	1    10400 1850
 	0    -1   -1   0
@@
 F 2 "Diode_SMD:D_SOD-123" H 10050 1650 50  0001 C CNN
 F 3 "~" H 10050 1650 50  0001 C CNN
+F 4 "C222352" H 10050 1650 50  0001 C CNN "LCSC"
 	1    10050 1650
 	0    1    1    0
@@
 F 2 "Capacitor_SMD:C_0603_1608Metric" H 2838 6650 50  0001 C CNN
 F 3 "~" H 2800 6800 50  0001 C CNN
+F 4 "C77055" H 2800 6800 50  0001 C CNN "LCSC"
 	1    2800 6800
 	1    0    0    -1
@@
 F 2 "Capacitor_SMD:C_1206_3216Metric" H 3688 6650 50  0001 C CNN
 F 3 "~" H 3650 6800 50  0001 C CNN
+F 4 "C14860" H 3650 6800 50  0001 C CNN "LCSC"
 	1    3650 6800
 	1    0    0    -1
@@
 F 0 "U2" H 3675 2281 50  0000 C CNN
 F 1 "PCA9557" H 3675 2190 50  0000 C CNN
-F 2 "Package_SO:SOIC-16_3.9x9.9mm_P1.27mm" H 3650 2050 50  0001 C CNN
+F 2 "Package_SO:TSSOP-16_4.4x5mm_P0.65mm" H 3650 2050 50  0001 C CNN
 F 3 "" H 3650 2050 50  0001 C CNN
+F 4 "C141380" H 3650 1650 50  0001 C CNN "LCSC"
 	1    3650 1650
 	1    0    0    -1
@@
 F 0 "R2" H 6320 1546 50  0000 L CNN
 F 1 "1k" H 6320 1455 50  0000 L CNN
-F 2 "Resistor_SMD:R_1206_3216Metric" V 6180 1500 50  0001 C CNN
+F 2 "Resistor_SMD:R_0603_1608Metric" V 6180 1500 50  0001 C CNN
 F 3 "~" H 6250 1500 50  0001 C CNN
+F 4 "C50069" H 6250 1500 50  0001 C CNN "LCSC"
 	1    6250 1500
 	1    0    0    -1
@@
 F 2 "LED_SMD:LED_1206_3216Metric" H 6250 1800 50  0001 C CNN
 F 3 "~" H 6250 1800 50  0001 C CNN
+F 4 "C264549" H 6250 1800 50  0001 C CNN "LCSC"
 	1    6250 1800
 	0    -1   -1   0
@@
 F 0 "R6" H 4320 1296 50  0000 L CNN
 F 1 "10k" H 4320 1205 50  0000 L CNN
-F 2 "Resistor_SMD:R_1206_3216Metric" V 4180 1250 50  0001 C CNN
+F 2 "Resistor_SMD:R_0603_1608Metric" V 4180 1250 50  0001 C CNN
 F 3 "~" H 4250 1250 50  0001 C CNN
+F 4 "C491175" H 4250 1250 50  0001 C CNN "LCSC"
 	1    4250 1250
 	1    0    0    -1
@@
 F 0 "R7" H 4570 1296 50  0000 L CNN
 F 1 "10k" H 4570 1205 50  0000 L CNN
-F 2 "Resistor_SMD:R_1206_3216Metric" V 4430 1250 50  0001 C CNN
+F 2 "Resistor_SMD:R_0603_1608Metric" V 4430 1250 50  0001 C CNN
 F 3 "~" H 4500 1250 50  0001 C CNN
+F 4 "C491175" H 4500 1250 50  0001 C CNN "LCSC"
 	1    4500 1250
 	1    0    0    -1
@@
 F 0 "R8" H 4820 1296 50  0000 L CNN
 F 1 "10k" H 4820 1205 50  0000 L CNN
-F 2 "Resistor_SMD:R_1206_3216Metric" V 4680 1250 50  0001 C CNN
+F 2 "Resistor_SMD:R_0603_1608Metric" V 4680 1250 50  0001 C CNN
 F 3 "~" H 4750 1250 50  0001 C CNN
+F 4 "C491175" H 4750 1250 50  0001 C CNN "LCSC"
 	1    4750 1250
 	1    0    0    -1
@@
 F 0 "R9" H 5070 1296 50  0000 L CNN
 F 1 "10k" H 5070 1205 50  0000 L CNN
-F 2 "Resistor_SMD:R_1206_3216Metric" V 4930 1250 50  0001 C CNN
+F 2 "Resistor_SMD:R_0603_1608Metric" V 4930 1250 50  0001 C CNN
 F 3 "~" H 5000 1250 50  0001 C CNN
+F 4 "C491175" H 5000 1250 50  0001 C CNN "LCSC"
 	1    5000 1250
 	1    0    0    -1
@@
 Wire Wire Line
 	5000 2100 5000 1400
+$Comp
+L Transistor_FET:BSS84 Q2
+U 1 1 5F26623C
+P 7250 1200
+F 0 "Q2" H 7454 1154 50  0000 L CNN
+F 1 "BSS84" H 7454 1245 50  0000 L CNN
+F 2 "Package_TO_SOT_SMD:SOT-23" H 7450 1125 50  0001 L CIN
+F 3 "http://assets.nexperia.com/documents/data-sheet/BSS84.pdf" H 7250 1200 50  0001 L CNN
+F 4 "C508197" H 7250 1200 50  0001 C CNN "LCSC"
+	1    7250 1200
+	1    0    0    1
+$EndComp
 $EndSCHEMATC
