File: spaceduino/spaceduino.kicad_pcb (KiCad board)
At the start: 2 copper layers, 69 x 69 mm, 72 parts, among them J1 USB_B, J3 JICSP, J4 Conn_02x05_Odd_Even, Q1 BSS84, Q2 BSS84, Q3 BSS84, SW1 SW_SPST, U1 TLV70030_SOT23-5, U2 FT230XS, U3 TXB0104D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

Commit message: some lcsc stuff
Parts:
- added C21: 100uF, Capacitor_THT:C_Radial_D5.0mm_H11.0mm_P2.00mm, B.Cu at (76.0, 84.0)
- added D3: LED, LED_SMD:LED_1206_3216Metric, B.Cu at (118.5, 110.5)
- added L3: 10uH, Inductor_SMD:L_1210_3225Metric, B.Cu at (113.5, 116.0)
- added R21: 10k, Resistor_SMD:R_1206_3216Metric, B.Cu at (101.6, 113.0)
- moved L2 2.55 mm to (114.5, 111.0), turned to 180 degrees
- moved DBPWR1 0.56 mm to (116.0, 106.5)
Connections:
- DBPWR1 pad 1: GND -> Net-(D3-Pad2)
- L2 pad 1: Net-(D2-Pad2) -> Net-(L2-Pad1)
Routing:
- net GND: track 157.1 -> 163.9 mm
- net 2_boost_en: track 23.9 -> 29.6 mm
- net Net-(L2-Pad1): track 0.00 -> 4.59 mm
- net Net-(D3-Pad2): track 0.00 -> 3.06 mm
- net +5V: track 21.1 -> 23.5 mm
- net Net-(D2-Pad2): track 6.26 -> 5.39 mm
