File: spaceduino/spaceduino.sch (KiCad schematic (older format))
At the start: 72 parts, among them J1 USB_B, J3 JICSP, J4 Conn_02x05_Odd_Even, Q1 BSS84, Q2 BSS84, Q3 BSS84, SW1 SW_SPST, U1 TLV70030_SOT23-5, U2 FT230XS, U3 TXB0104D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

Commit message: some lcsc stuff
Parts:
- added C21: 100uF, Capacitor_THT:C_Radial_D5.0mm_H11.0mm_P2.00mm, symbol Device:C
- added DBPWR2: LED, LED_SMD:LED_1206_3216Metric, symbol Device:LED
- added L3: 10uH, Inductor_SMD:L_1210_3225Metric, symbol Device:L
- added R21: 10k, Resistor_SMD:R_1206_3216Metric, symbol Device:R
- C1, C10, C12, C16, C19, C2, C20, C3, C5, C9: Comment (none) -> .1uF; LCSC (none) -> C77055
- C11, C13: Comment (none) -> 22pF; LCSC (none) -> C599690
- C14, C17, C8: Comment (none) -> 10uF; LCSC (none) -> C14860
- C15: Comment (none) -> 1.5nF; LCSC (none) -> C519421
- C18: footprint Capacitor_SMD:C_0603_1608Metric -> Capacitor_SMD:C_1206_3216Metric; Comment (none) -> 10uF; LCSC (none) -> C14860
- C4: Comment (none) -> 1uF; LCSC (none) -> C141215
- C6, C7: Comment (none) -> 47pF; LCSC (none) -> C1671
- D2: LCSC (none) -> C222352
- D3PWR1, DALERT1, DBPWR1, DIND1, DPWR1: LCSC (none) -> C192676
- F1: LCSC (none) -> C315895
- FB1: LCSC (none) -> C88995
- L1: value L -> 10uH; Comment (none) -> 10uH; LCSC (none) -> C86073
- L2: Comment (none) -> 10uH; LCSC (none) -> C86073
- MICROSD1: footprint Connector_Card:microSD_HC_Hirose_DM3D-SF -> Spaceduino:HRS_DM3CS-SF; LCSC (none) -> C202111
- Q1, Q2, Q3: LCSC (none) -> C508197
- R1, R2: Comment (none) -> 1K; LCSC (none) -> C52199
- R10: Comment (none) -> 36K; LCSC (none) -> C18007
- R11, R6: Comment (none) -> 50mR
- R12, R15, R16, R9: Comment (none) -> 1.5K; LCSC (none) -> C26030
- R13: Comment (none) -> 470R; LCSC (none) -> C4502
- R14: Comment (none) -> 5K6; LCSC (none) -> C18028
- R17, R18: Comment (none) -> 3K3; LCSC (none) -> C26032
- R19, R20: Comment (none) -> 100R; LCSC (none) -> C17901
- R3, R4: Comment (none) -> 27R; LCSC (none) -> C17946
- R5, R8: Comment (none) -> 10K; LCSC (none) -> C17902
- R7: Comment (none) -> 13K; LCSC (none) -> C34847
- U1: LCSC (none) -> C36463
- U2: LCSC (none) -> C69082
- U3: footprint Package_SO:SOIC-14_3.9x8.7mm_P1.27mm -> Package_SO:TSSOP-14_4.4x5mm_P0.65mm; LCSC (none) -> C60708
- U6: LCSC (none) -> C33575
Connections:
- net +5V: now also C21.1
- net 2_boost_en: now also R21.1
- net GND: now also C21.2, DBPWR2.1 (K), R21.2; no longer DBPWR1.1 (K)
- net at D2.2 (A), U4.1 (SW): now also L3.1; no longer L2.1
- new net: DBPWR1.1 (K), DBPWR2.2 (A)
- new net: L2.1, L3.2
Other:
- note added: "both blue/white, or zener & led"
- moved on the sheet: DALERT1, DBPWR1, DIND1, L2, R14, R15, R16

Commit message: more lcsc, redo a lot of inner containment
Parts:
- D1: LCSC (none) -> C222352
- DBPWR1, DBPWR2: LCSC C192676 -> C264549
- R11, R6: LCSC (none) -> C601102
- U4: LCSC (none) -> C32355
Changed lines of the file:
@@
 F 2 "Package_TO_SOT_SMD:SOT-23-5" H 1450 3700 50  0001 L CIN
 F 3 "http://www.ti.com/lit/ds/symlink/lm27313.pdf" H 1400 4050 50  0001 C CNN
+F 4 "C32355" H 1400 3950 50  0001 C CNN "LCSC"
 	1    1400 3950
 	1    0    0    -1
@@
 F 3 "~" H 7850 4850 50  0001 C CNN
 F 4 "50mR" H 7850 4850 50  0001 C CNN "Comment"
+F 5 "C601102" H 7850 4850 50  0001 C CNN "LCSC"
 	1    7850 4850
 	0    1    1    0
@@
 F 2 "Diode_SMD:D_SOD-123" H 4700 3000 50  0001 C CNN
 F 3 "~" H 4700 3000 50  0001 C CNN
+F 4 "C222352" H 4700 3000 50  0001 C CNN "LCSC"
 	1    4700 3000
 	0    1    1    0
@@
 F 3 "~" H 3200 3300 50  0001 C CNN
 F 4 "50mR" H 3200 3300 50  0001 C CNN "Comment"
+F 5 "C601102" H 3200 3300 50  0001 C CNN "LCSC"
 	1    3200 3300
 	0    1    1    0
@@
 F 2 "LED_SMD:LED_1206_3216Metric" H 1700 5550 50  0001 C CNN
 F 3 "~" H 1700 5550 50  0001 C CNN
-F 4 "C192676" H 1700 5550 50  0001 C CNN "LCSC"
+F 4 "C264549" H 1700 5550 50  0001 C CNN "LCSC"
 	1    1700 5550
 	0    -1   -1   0
@@
 F 2 "LED_SMD:LED_1206_3216Metric" H 1700 5850 50  0001 C CNN
 F 3 "~" H 1700 5850 50  0001 C CNN
-F 4 "C192676" H 1700 5850 50  0001 C CNN "LCSC"
+F 4 "C264549" H 1700 5850 50  0001 C CNN "LCSC"
 	1    1700 5850
 	0    -1   -1   0
